Commit message: M4: MuJoCo plant behind ros2_control (topic_based_ros2_control); JTC tolerances
- ex_mujoco_sim: URDF->MJCF at runtime from the same robot_description (FK matches URDF to ~1.5 um),
  explicit dynamics assumptions, servo-drive model (kp=M w^2, kd=2 zeta M w, FOH set-point
  interpolation, gravity/Coriolis feedforward, torque limits), 1 kHz real-time paced, 500 Hz states
- sim_moveit.launch.py plant:=mock|mujoco (+payload_kg, bandwidth_hz, mujoco_viewer); M2 tools unchanged
- fixes found on the way: thread-local 'import mujoco.viewer' shadowing (UnboundLocalError) left a
  healthy-looking node with a dead physics thread -> crash now terminates the node; JTC without
  per-joint tolerances reported SUCCESS for a plant that never moved -> goal/trajectory tolerances
- scripts/setup_mujoco.sh (offline, keeps system numpy 1.21); 12 new unit tests

Co-Authored-By: Claude Opus 5.5 <noreply@anthropic.com>

File: ros2_ws/src/ex_moveit_config/urdf/ex_cr10_moveit.urdf.xacro (robot description, xacro)
@@ -1,9 +1,13 @@
 <?xml version="1.0"?>
-<!-- CR10 model + ros2_control with mock_components/GenericSystem (SIMULATION ONLY).
+<!-- CR10 model + ros2_control hardware for SIMULATION ONLY.
+     arg plant:
+       mock    mock_components/GenericSystem: ideal position following, no dynamics (M2)
+       mujoco  topic_based_ros2_control/TopicBasedSystem <-> ex_mujoco_sim (physics plant, M4)
      There is deliberately no hardware plugin for a real Dobot controller in this package. -->
 <robot name="ex_cr10" xmlns:xacro="http://www.ros.org/wiki/xacro">
+  <xacro:arg name="plant" default="mock"/>
   <xacro:include filename="$(find ex_description)/urdf/ex_cr10.urdf.xacro"/>
   <xacro:property name="home" value="${[0.0, 0.0, pi/2, 0.0, -pi/2, 0.0]}"/>
-  <xacro:macro name="mock_joint" params="i">
+  <xacro:macro name="sim_joint" params="i">
     <joint name="joint${i}">
       <command_interface name="position"/>
@@ -12,15 +16,23 @@
     </joint>
   </xacro:macro>
-  <ros2_control name="MockCR10" type="system">
+  <ros2_control name="SimCR10" type="system">
     <hardware>
-      <plugin>mock_components/GenericSystem</plugin>
-      <param name="calculate_dynamics">true</param>
+      <xacro:if value="${'$(arg plant)' == 'mujoco'}">
+        <plugin>topic_based_ros2_control/TopicBasedSystem</plugin>
+        <param name="joint_commands_topic">/mujoco/joint_commands</param>
+        <param name="joint_states_topic">/mujoco/joint_states</param>
+        <param name="trigger_joint_command_threshold">-1</param>
+      </xacro:if>
+      <xacro:unless value="${'$(arg plant)' == 'mujoco'}">
+        <plugin>mock_components/GenericSystem</plugin>
+        <param name="calculate_dynamics">true</param>
+      </xacro:unless>
     </hardware>
-    <xacro:mock_joint i="1"/>
-    <xacro:mock_joint i="2"/>
-    <xacro:mock_joint i="3"/>
-    <xacro:mock_joint i="4"/>
-    <xacro:mock_joint i="5"/>
-    <xacro:mock_joint i="6"/>
+    <xacro:sim_joint i="1"/>
+    <xacro:sim_joint i="2"/>
+    <xacro:sim_joint i="3"/>
+    <xacro:sim_joint i="4"/>
+    <xacro:sim_joint i="5"/>
+    <xacro:sim_joint i="6"/>
   </ros2_control>
 </robot>
